File: Hardware/Layout/Marvin_0.5.2.brd (EAGLE design)
At the start: 85 x 30 mm, 56 parts, among them IC1 LM321MF, Q1 IRLML5203, Q2 IRLML5203, Q3 IRLML5203, U1 ATMEGA32U4-XUAU, U2 SI2366DS-T1-GE3, U3 SI2366DS-T1-GE3, U4 SI2366DS-T1-GE3, U5 LT1761IS5-3.3TRMPBF, X3 BU-SMA-H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

Commit message: pics
Routing:
- net RX: track 50.6 -> 47.2 mm
Changed lines of the file:
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@@
 <layer number="14" name="Route14" color="1" fill="6" visible="no" active="no"/>
 <layer number="15" name="Route15" color="4" fill="6" visible="no" active="no"/>
-<layer number="16" name="Bottom" color="1" fill="1" visible="no" active="yes"/>
+<layer number="16" name="Bottom" color="1" fill="1" visible="yes" active="yes"/>
 <layer number="17" name="Pads" color="2" fill="1" visible="yes" active="yes"/>
 <layer number="18" name="Vias" color="2" fill="1" visible="yes" active="yes"/>
@@
 <layer number="20" name="Dimension" color="15" fill="1" visible="yes" active="yes"/>
 <layer number="21" name="tPlace" color="7" fill="1" visible="yes" active="yes"/>
-<layer number="22" name="bPlace" color="7" fill="1" visible="no" active="yes"/>
-<layer number="23" name="tOrigins" color="15" fill="1" visible="no" active="yes"/>
-<layer number="24" name="bOrigins" color="15" fill="1" visible="no" active="yes"/>
+<layer number="22" name="bPlace" color="7" fill="1" visible="yes" active="yes"/>
+<layer number="23" name="tOrigins" color="15" fill="1" visible="yes" active="yes"/>
+<layer number="24" name="bOrigins" color="15" fill="1" visible="yes" active="yes"/>
 <layer number="25" name="tNames" color="7" fill="1" visible="no" active="yes"/>
 <layer number="26" name="bNames" color="7" fill="1" visible="no" active="yes"/>
@@
 <layer number="28" name="bValues" color="7" fill="1" visible="no" active="yes"/>
 <layer number="29" name="tStop" color="7" fill="3" visible="yes" active="yes"/>
-<layer number="30" name="bStop" color="7" fill="6" visible="no" active="yes"/>
+<layer number="30" name="bStop" color="7" fill="6" visible="yes" active="yes"/>
 <layer number="31" name="tCream" color="7" fill="4" visible="no" active="yes"/>
 <layer number="32" name="bCream" color="7" fill="5" visible="no" active="yes"/>
@@
 <layer number="50" name="dxf" color="7" fill="1" visible="no" active="no"/>
 <layer number="51" name="tDocu" color="7" fill="1" visible="yes" active="yes"/>
-<layer number="52" name="bDocu" color="7" fill="1" visible="no" active="yes"/>
+<layer number="52" name="bDocu" color="7" fill="1" visible="yes" active="yes"/>
 <layer number="53" name="tGND_GNDA" color="7" fill="9" visible="no" active="no"/>
 <layer number="54" name="bGND_GNDA" color="1" fill="9" visible="no" active="no"/>
@@
 <text x="20.7" y="18.6" size="0.9" layer="29" font="vector" ratio="10" rot="R180" align="center-left">ON</text>
 <text x="78.3" y="28.45" size="2.2" layer="29" font="vector" ratio="11" rot="SR0" align="top-center">Marvin</text>
-<text x="15.1" y="7.9" size="0.9" layer="29" font="vector" ratio="10" align="center-left">RESET</text>
+<text x="15.1" y="8" size="0.9" layer="29" font="vector" ratio="10" align="center-left">RESET</text>
 <wire x1="72.7" y1="25.8" x2="74.6" y2="25.8" width="0.3048" layer="29"/>
 <wire x1="74.6" y1="25.8" x2="76.6" y2="25.8" width="0.3048" layer="29"/>
@@
 <contactref element="U$16" pad="P$1"/>
 <via x="17.5" y="18.3" extent="1-16" drill="0.3"/>
-<via x="15.8" y="7.8" extent="1-16" drill="0.3"/>
+<via x="15.8" y="4.6" extent="1-16" drill="0.3"/>
 <via x="39.35" y="8.85" extent="1-16" drill="0.3"/>
 <contactref element="R8" pad="2"/>
@@
 <wire x1="45.5" y1="5" x2="44.8" y2="5" width="0.254" layer="1"/>
 <contactref element="Q2" pad="1"/>
-<via x="17.25" y="8.3" extent="1-16" drill="0.3"/>
+<via x="18.85" y="6.75" extent="1-16" drill="0.3"/>
 <wire x1="19.5" y1="3.25" x2="40" y2="3.2" width="0.254" layer="16"/>
 <wire x1="40" y1="3.2" x2="40.2" y2="3" width="0.254" layer="16"/>
@@
 <wire x1="23.25" y1="8.85" x2="23.25" y2="8.5" width="0.3048" layer="1"/>
 <wire x1="23.25" y1="8.5" x2="22.7" y2="7.95" width="0.3048" layer="1"/>
-<wire x1="22.7" y1="7.95" x2="17.6" y2="7.95" width="0.3048" layer="1"/>
-<wire x1="17.6" y1="7.95" x2="17.25" y2="8.3" width="0.3048" layer="1"/>
-<wire x1="19.5" y1="3.25" x2="17.25" y2="5.5" width="0.3048" layer="16"/>
-<wire x1="17.25" y1="5.5" x2="17.25" y2="8.3" width="0.3048" layer="16"/>
+<wire x1="22.7" y1="7.95" x2="20.05" y2="7.95" width="0.3048" layer="1"/>
+<wire x1="20.05" y1="7.95" x2="18.85" y2="6.75" width="0.3048" layer="1"/>
+<wire x1="19.5" y1="3.25" x2="18.85" y2="3.9" width="0.3048" layer="16"/>
+<wire x1="18.85" y1="3.9" x2="18.85" y2="6.75" width="0.3048" layer="16"/>
 </signal>
 <signal name="RFH">

Commit message: brd updates
Parts:
- moved R13 0.20 mm to (47.9, 2.90)
- moved ON 0.10 mm to (19.8, 16.5)
- moved R2 0.10 mm to (19.8, 13.7)
- moved Y1 0.10 mm to (38.8, 2.70)
Routing:
- net TX: track 53.2 -> 52.6 mm
- net A6: track 17.4 -> 18.0 mm
- net GND: vias 53 -> 52
Other:
- outline, holes or cut-outs redrawn

Commit message: cleaning up pcb
Parts:
- removed X3: BU-SMA-H, con-coax:BU-SMA-H
- added U$25: 868AT, 868AT43_antenna:868AT
Connections:
- new net N$13: U$25.2
- net GND: no longer X3.2, X3.3, X3.4, X3.5
- net RFH: now also U$25.1; no longer X3.1
Routing:
- net N$12: track 0.00 -> 18.4 mm
- net GND: track 17.4 -> 21.4 mm, vias 52 -> 39
- net RFH: track 7.09 -> 3.45 mm
- net +5V: track 211.0 -> 209.3 mm
Other:
- board text removed: "Academy"
- board text removed: "IoT"
