File: Hardware/Layout/Marvin_1.0.sch (EAGLE design)
At the start: 56 parts, among them IC1 LM321MF, Q1 IRLML5203, Q2 IRLML5203, Q3 IRLML5203, U1 ATMEGA32U4-XUAU, U2 SI2366DS-T1-GE3, U3 SI2366DS-T1-GE3, U4 SI2366DS-T1-GE3, U5 LT1761IS5-3.3TRMPBF, Y1 CSTCE16M0V53-R0 16MHZ

Commit message: pics
Parts:
- removed U2, U3, U4: SI2366DS-T1-GE3, Vishay_By_element14_Batch_1:SI2366DS-T1-GE3
- added Q4, Q5, Q6: BSS138, m-pad-2.1:BSS138
- R8: value 100k -> 10k
Connections:
- removed net RN_RX: R3.1, U$1.UART_RX, U3.S
- removed net RN_TX: R12.1, U$1.UART_TX, U4.S
- removed net RX: PAD2.P, Q2.G, R13.1, TP8.TP, U1.(RXD1/AIN1/INT2)PD2, U4.D
- removed net TX: PAD1.P, Q3.G, R11.1, TP7.TP, U1.(TXD1/INT3)PD3, U3.D
- new net ATMEGA_RX: PAD2.P, Q2.G, Q4.D, R13.1, TP8.TP, U1.(RXD1/AIN1/INT2)PD2
- new net ATMEGA_TX: PAD1.P, Q3.G, Q5.D, R11.1, TP7.TP, U1.(TXD1/INT3)PD3
- new net RN2483_RX: Q5.S, R3.1, U$1.UART_RX
- new net RN2483_TX: Q4.S, R12.1, U$1.UART_TX
- net +3V3: now also Q4.G, Q5.G, Q6.G; no longer U2.G, U3.G, U4.G
- net LORA_RESET_33V: now also Q6.S; no longer U2.S
- net LORA_RESET_5V: now also Q6.D; no longer U2.D
Other:
- note removed: "Antenna"
- moved on the sheet: R11, R12, R13, R14, R3, R9

Commit message: intro
Connections:
- net N$5 renamed L_ON
- net N$6 renamed POWERLED
Changed lines of the file:
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@@
 <part name="GND12" library="supply1" deviceset="GND" device=""/>
 <part name="GND13" library="supply1" deviceset="GND" device=""/>
-<part name="GND14" library="supply1" deviceset="GND" device=""/>
-<part name="GND15" library="supply1" deviceset="GND" device=""/>
-<part name="GND16" library="supply1" deviceset="GND" device=""/>
-<part name="GND17" library="supply1" deviceset="GND" device=""/>
 <part name="GND18" library="supply1" deviceset="GND" device=""/>
 <part name="GND19" library="supply1" deviceset="GND" device=""/>
@@
 <instance part="GND11" gate="1" x="274.32" y="271.78" rot="R90"/>
 <instance part="GND12" gate="1" x="274.32" y="294.64" rot="R90"/>
-<instance part="GND13" gate="1" x="254" y="314.96" rot="R180"/>
-<instance part="GND14" gate="1" x="251.46" y="314.96" rot="R180"/>
-<instance part="GND15" gate="1" x="246.38" y="314.96" rot="R180"/>
-<instance part="GND16" gate="1" x="241.3" y="314.96" rot="R180"/>
-<instance part="GND17" gate="1" x="238.76" y="314.96" rot="R180"/>
+<instance part="GND13" gate="1" x="256.54" y="312.42" rot="R90"/>
 <instance part="GND18" gate="1" x="218.44" y="294.64" rot="R270"/>
 <instance part="GND19" gate="1" x="218.44" y="281.94" rot="R270"/>
@@
 </segment>
 <segment>
+<pinref part="U$1" gate="G$1" pin="GND27"/>
+<pinref part="U$1" gate="G$1" pin="GND26"/>
+<wire x1="238.76" y1="312.42" x2="241.3" y2="312.42" width="0.1524" layer="91"/>
+<junction x="241.3" y="312.42"/>
+<pinref part="U$1" gate="G$1" pin="GND24"/>
+<wire x1="241.3" y1="312.42" x2="246.38" y2="312.42" width="0.1524" layer="91"/>
+<junction x="246.38" y="312.42"/>
+<pinref part="U$1" gate="G$1" pin="GND22"/>
+<wire x1="246.38" y1="312.42" x2="251.46" y2="312.42" width="0.1524" layer="91"/>
+<junction x="251.46" y="312.42"/>
 <pinref part="U$1" gate="G$1" pin="GND21"/>
 <pinref part="GND13" gate="1" pin="GND"/>
-</segment>
-<segment>
-<pinref part="U$1" gate="G$1" pin="GND22"/>
-<pinref part="GND14" gate="1" pin="GND"/>
-</segment>
-<segment>
-<pinref part="U$1" gate="G$1" pin="GND24"/>
-<pinref part="GND15" gate="1" pin="GND"/>
-</segment>
-<segment>
-<pinref part="U$1" gate="G$1" pin="GND26"/>
-<pinref part="GND16" gate="1" pin="GND"/>
-</segment>
-<segment>
-<pinref part="U$1" gate="G$1" pin="GND27"/>
-<pinref part="GND17" gate="1" pin="GND"/>
+<wire x1="251.46" y1="312.42" x2="254" y2="312.42" width="0.1524" layer="91"/>
+<junction x="254" y="312.42"/>
+<junction x="238.76" y="312.42"/>
 </segment>
 <segment>
@@
 </segment>
 </net>
-<net name="N$5" class="0">
+<net name="L_ON" class="0">
 <segment>
 <pinref part="U1" gate="G$1" pin="(ICP3/CLK0/OC4A)PC7"/>
@@
 <wire x1="193.04" y1="68.58" x2="157.48" y2="68.58" width="0.1524" layer="91"/>
 <pinref part="IC1" gate="G$1" pin="+IN"/>
+<label x="170.18" y="68.58" size="1.778" layer="95"/>
 </segment>
 </net>
@@
 </segment>
 </net>
-<net name="N$6" class="0">
+<net name="POWERLED" class="0">
 <segment>
 <pinref part="U5" gate="A" pin="~SHDN"/>
@@
 <pinref part="R1" gate="G$1" pin="1"/>
 <junction x="210.82" y="25.4"/>
-</segment>
-</net>
+<label x="170.18" y="53.34" size="1.778" layer="95"/>
+</segment>
+</net>
